Commit message: update: gemini 336에 맞춰 camera_link 추가

File: nero/urdf/nero_with_handeye_description.xacro (robot description, xacro)
@@ -111,5 +111,5 @@
   </joint>
   <link
-    name="hand_eye_camera_link">
+    name="hand_eye_camera_base_link">
     <inertial>
       <origin
@@ -159,7 +159,13 @@
       link="endeffector_base_link" />
     <child
-      link="hand_eye_camera_link" />
+      link="hand_eye_camera_base_link" />
     <axis
       xyz="0 0 0" />
   </joint>
+  <link name="camera_link"/>
+  <joint name="camera_internal_joint" type="fixed">
+    <parent link="hand_eye_camera_base_link"/>
+    <child link="camera_link"/>
+    <origin xyz="0.01587 0.025 0.0125" rpy="0 0 0"/>
+  </joint>
 </robot>
